File: Board Files/Breadboard_DMM/Level Shifter.sch (KiCad schematic (older format))
At the start: 6 parts, among them Q1001 NTZD3154N, Q801 NTZD3154N

Commit message: Started adding Digikey links
Parts:
- Q1001, Q801: Digi-Key Link (none) -> https://www.digikey.com/en/products/detail/on-semiconductor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; Digi-Key PN - -> NTZD3154NT1GOSCT-ND
Changed lines of the file:
@@
 $Descr A4 11693 8268
 encoding utf-8
-Sheet 10 10
+Sheet 10 11
 Title "Toast-O-Meter"
-Date ""
+Date "2020-08-14"
 Rev "0"
 Comp ""
@@
 F 2 "Package_TO_SOT_SMD:SOT-563" H 5850 3450 50  0001 L CNN
 F 3 "https://www.onsemi.cn/PowerSolutions/document/NTZD3154N-D.PDF" H 5750 3550 50  0001 L CNN
-F 4 "" H 5750 3550 50  0001 C CNN "Digi-Key Link"
-F 5 "-" H 5750 3550 50  0001 C CNN "Digi-Key PN"
+F 4 "https://www.digikey.com/en/products/detail/on-semiconductor/NTZD3154NT1G/687137" H 5750 3550 50  0001 C CNN "Digi-Key Link"
+F 5 "NTZD3154NT1GOSCT-ND" H 5750 3550 50  0001 C CNN "Digi-Key PN"
 	2    5750 3550
 	0    1    1    0
@@
 F 2 "Package_TO_SOT_SMD:SOT-563" H 5850 4900 50  0001 L CNN
 F 3 "https://www.onsemi.cn/PowerSolutions/document/NTZD3154N-D.PDF" H 5750 5000 50  0001 L CNN
-F 4 "" H 5750 5000 50  0001 C CNN "Digi-Key Link"
-F 5 "-" H 5750 5000 50  0001 C CNN "Digi-Key PN"
+F 4 "https://www.digikey.com/en/products/detail/on-semiconductor/NTZD3154NT1G/687137" H 5750 5000 50  0001 C CNN "Digi-Key Link"
+F 5 "NTZD3154NT1GOSCT-ND" H 5750 5000 50  0001 C CNN "Digi-Key PN"
 	1    5750 5000
 	0    1    1    0
