File: Board Files/Breadboard_DMM/user_input.sch (KiCad schematic (older format))
At the start: 12 parts, among them SW1101 SW_Push, SW1102 SW_Push, SW1103 SW_Push

Commit message: Finished adding parts, cleaned up, ran ERC
Parts:
- C1101, C1102, C1103: footprint (none) -> Resistor_SMD:R_0603_1608Metric_Pad1.05x0.95mm_HandSolder; Digi-Key Link (none) -> https://www.digikey.com/en/products/detail/samsung-electro-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; Digi-Key PN - -> 1276-1006-1-ND
- R1101: footprint (none) -> Resistor_SMD:R_0603_1608Metric_Pad1.05x0.95mm_HandSolder; Digi-Key Link (none) -> https://www.digikey.com/en/products/detail/yageo/RC0603FR-0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; Digi-Key PN - -> 311-10.0KHRCT-ND
- R1102: renamed from R1103; footprint (none) -> Resistor_SMD:R_0603_1608Metric_Pad1.05x0.95mm_HandSolder; Digi-Key Link (none) -> https://www.digikey.com/en/products/detail/yageo/RC0603FR-0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; Digi-Key PN - -> 311-10.0KHRCT-ND
- R1103: renamed from R1105; footprint (none) -> Resistor_SMD:R_0603_1608Metric_Pad1.05x0.95mm_HandSolder; Digi-Key Link (none) -> https://www.digikey.com/en/products/detail/yageo/RC0603FR-0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; Digi-Key PN - -> 311-10.0KHRCT-ND
- R1104: renamed from R1102; footprint (none) -> Resistor_SMD:R_0603_1608Metric_Pad1.05x0.95mm_HandSolder; Digi-Key Link (none) -> https://www.digikey.com/en/products/detail/yageo/RC0603FR-0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; Digi-Key PN - -> 311-1.00KHRCT-ND
- R1105: renamed from R1104; footprint (none) -> Resistor_SMD:R_0603_1608Metric_Pad1.05x0.95mm_HandSolder; Digi-Key Link (none) -> https://www.digikey.com/en/products/detail/yageo/RC0603FR-0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; Digi-Key PN - -> 311-1.00KHRCT-ND
- R1106: footprint (none) -> Resistor_SMD:R_0603_1608Metric_Pad1.05x0.95mm_HandSolder; Digi-Key Link (none) -> https://www.digikey.com/en/products/detail/yageo/RC0603FR-0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; Digi-Key PN - -> 311-1.00KHRCT-ND
Changed lines of the file:
@@
 P 3900 3650
 AR Path="/5F3FD151/5F83BFE2" Ref="R?"  Part="1"
-AR Path="/5F3FD151/5F82FB20/5F83BFE2" Ref="R1103"  Part="1"
-F 0 "R1103" H 3968 3696 50  0000 L CNN
+AR Path="/5F3FD151/5F82FB20/5F83BFE2" Ref="R1102"  Part="1"
+F 0 "R1102" H 3968 3696 50  0000 L CNN
 F 1 "10k" H 3968 3605 50  0000 L CNN
-F 2 "" V 3940 3640 50  0001 C CNN
+F 2 "Resistor_SMD:R_0603_1608Metric_Pad1.05x0.95mm_HandSolder" V 3940 3640 50  0001 C CNN
 F 3 "~" H 3900 3650 50  0001 C CNN
-F 4 "" H 3900 3650 50  0001 C CNN "Digi-Key Link"
-F 5 "-" H 3900 3650 50  0001 C CNN "Digi-Key PN"
+F 4 "https://www.digikey.com/en/products/detail/yageo/RC0603FR-0710KL/726880?s=N4IgTCBcDaIEoGEAMA2JBmAYnAtEg7AIxIDSAMiALoC%2BQA" H 3900 3650 50  0001 C CNN "Digi-Key Link"
+F 5 "311-10.0KHRCT-ND" H 3900 3650 50  0001 C CNN "Digi-Key PN"
 	1    3900 3650
 	1    0    0    -1
@@
 P 5100 4550
 AR Path="/5F3FD151/5F83BFE8" Ref="#PWR?"  Part="1"
-AR Path="/5F3FD151/5F82FB20/5F83BFE8" Ref="#PWR01106"  Part="1"
-F 0 "#PWR01106" H 5100 4300 50  0001 C CNN
+AR Path="/5F3FD151/5F82FB20/5F83BFE8" Ref="#PWR01108"  Part="1"
+F 0 "#PWR01108" H 5100 4300 50  0001 C CNN
 F 1 "GND" H 5105 4377 50  0000 C CNN
 F 2 "" H 5100 4550 50  0001 C CNN
@@
 F 0 "C1102" H 4215 4296 50  0000 L CNN
 F 1 "0.1uF" H 4215 4205 50  0000 L CNN
-F 2 "" H 4138 4100 50  0001 C CNN
+F 2 "Resistor_SMD:R_0603_1608Metric_Pad1.05x0.95mm_HandSolder" H 4138 4100 50  0001 C CNN
 F 3 "~" H 4100 4250 50  0001 C CNN
-F 4 "" H 4100 4250 50  0001 C CNN "Digi-Key Link"
-F 5 "-" H 4100 4250 50  0001 C CNN "Digi-Key PN"
+F 4 "https://www.digikey.com/en/products/detail/samsung-electro-mechanics/CL10B104KA8NNNC/3886664" H 4100 4250 50  0001 C CNN "Digi-Key Link"
+F 5 "1276-1006-1-ND" H 4100 4250 50  0001 C CNN "Digi-Key PN"
 	1    4100 4250
 	1    0    0    -1
@@
 P 5100 4300
 AR Path="/5F3FD151/5F83C001" Ref="R?"  Part="1"
-AR Path="/5F3FD151/5F82FB20/5F83C001" Ref="R1104"  Part="1"
-F 0 "R1104" H 5168 4346 50  0000 L CNN
+AR Path="/5F3FD151/5F82FB20/5F83C001" Ref="R1105"  Part="1"
+F 0 "R1105" H 5168 4346 50  0000 L CNN
 F 1 "1k" H 5168 4255 50  0000 L CNN
-F 2 "" V 5140 4290 50  0001 C CNN
+F 2 "Resistor_SMD:R_0603_1608Metric_Pad1.05x0.95mm_HandSolder" V 5140 4290 50  0001 C CNN
 F 3 "~" H 5100 4300 50  0001 C CNN
-F 4 "" H 5100 4300 50  0001 C CNN "Digi-Key Link"
-F 5 "-" H 5100 4300 50  0001 C CNN "Digi-Key PN"
+F 4 "https://www.digikey.com/en/products/detail/yageo/RC0603FR-071KL/726843" H 5100 4300 50  0001 C CNN "Digi-Key Link"
+F 5 "311-1.00KHRCT-ND" H 5100 4300 50  0001 C CNN "Digi-Key PN"
 	1    5100 4300
 	1    0    0    -1
@@
 P 3900 3400
 AR Path="/5F3FD151/5F83C00F" Ref="#PWR?"  Part="1"
-AR Path="/5F3FD151/5F82FB20/5F83C00F" Ref="#PWR01104"  Part="1"
-F 0 "#PWR01104" H 3900 3250 50  0001 C CNN
+AR Path="/5F3FD151/5F82FB20/5F83C00F" Ref="#PWR01102"  Part="1"
+F 0 "#PWR01102" H 3900 3250 50  0001 C CNN
 F 1 "+3V3" H 3915 3573 50  0000 C CNN
 F 2 "" H 3900 3400 50  0001 C CNN
@@
 P 3900 5850
 AR Path="/5F3FD151/5F841C24" Ref="R?"  Part="1"
-AR Path="/5F3FD151/5F82FB20/5F841C24" Ref="R1105"  Part="1"
-F 0 "R1105" H 3968 5896 50  0000 L CNN
+AR Path="/5F3FD151/5F82FB20/5F841C24" Ref="R1103"  Part="1"
+F 0 "R1103" H 3968 5896 50  0000 L CNN
 F 1 "10k" H 3968 5805 50  0000 L CNN
-F 2 "" V 3940 5840 50  0001 C CNN
+F 2 "Resistor_SMD:R_0603_1608Metric_Pad1.05x0.95mm_HandSolder" V 3940 5840 50  0001 C CNN
 F 3 "~" H 3900 5850 50  0001 C CNN
-F 4 "" H 3900 5850 50  0001 C CNN "Digi-Key Link"
-F 5 "-" H 3900 5850 50  0001 C CNN "Digi-Key PN"
+F 4 "https://www.digikey.com/en/products/detail/yageo/RC0603FR-0710KL/726880?s=N4IgTCBcDaIEoGEAMA2JBmAYnAtEg7AIxIDSAMiALoC%2BQA" H 3900 5850 50  0001 C CNN "Digi-Key Link"
+F 5 "311-10.0KHRCT-ND" H 3900 5850 50  0001 C CNN "Digi-Key PN"
 	1    3900 5850
 	1    0    0    -1
@@
 F 0 "C1103" H 4215 6496 50  0000 L CNN
 F 1 "0.1uF" H 4215 6405 50  0000 L CNN
-F 2 "" H 4138 6300 50  0001 C CNN
+F 2 "Resistor_SMD:R_0603_1608Metric_Pad1.05x0.95mm_HandSolder" H 4138 6300 50  0001 C CNN
 F 3 "~" H 4100 6450 50  0001 C CNN
-F 4 "" H 4100 6450 50  0001 C CNN "Digi-Key Link"
-F 5 "-" H 4100 6450 50  0001 C CNN "Digi-Key PN"
+F 4 "https://www.digikey.com/en/products/detail/samsung-electro-mechanics/CL10B104KA8NNNC/3886664" H 4100 6450 50  0001 C CNN "Digi-Key Link"
+F 5 "1276-1006-1-ND" H 4100 6450 50  0001 C CNN "Digi-Key PN"
 	1    4100 6450
 	1    0    0    -1
@@
 P 4100 6750
 AR Path="/5F3FD151/5F841C46" Ref="#PWR?"  Part="1"
-AR Path="/5F3FD151/5F82FB20/5F841C46" Ref="#PWR01108"  Part="1"
-F 0 "#PWR01108" H 4100 6500 50  0001 C CNN
+AR Path="/5F3FD151/5F82FB20/5F841C46" Ref="#PWR01106"  Part="1"
+F 0 "#PWR01106" H 4100 6500 50  0001 C CNN
 F 1 "GND" H 4105 6577 50  0000 C CNN
 F 2 "" H 4100 6750 50  0001 C CNN
@@
 F 0 "R1106" H 5168 6546 50  0000 L CNN
 F 1 "1k" H 5168 6455 50  0000 L CNN
-F 2 "" V 5140 6490 50  0001 C CNN
+F 2 "Resistor_SMD:R_0603_1608Metric_Pad1.05x0.95mm_HandSolder" V 5140 6490 50  0001 C CNN
 F 3 "~" H 5100 6500 50  0001 C CNN
-F 4 "" H 5100 6500 50  0001 C CNN "Digi-Key Link"
-F 5 "-" H 5100 6500 50  0001 C CNN "Digi-Key PN"
+F 4 "https://www.digikey.com/en/products/detail/yageo/RC0603FR-071KL/726843" H 5100 6500 50  0001 C CNN "Digi-Key Link"
+F 5 "311-1.00KHRCT-ND" H 5100 6500 50  0001 C CNN "Digi-Key PN"
 	1    5100 6500
 	1    0    0    -1
@@
 P 3900 5600
 AR Path="/5F3FD151/5F841C64" Ref="#PWR?"  Part="1"
-AR Path="/5F3FD151/5F82FB20/5F841C64" Ref="#PWR01107"  Part="1"
-F 0 "#PWR01107" H 3900 5450 50  0001 C CNN
+AR Path="/5F3FD151/5F82FB20/5F841C64" Ref="#PWR01103"  Part="1"
+F 0 "#PWR01103" H 3900 5450 50  0001 C CNN
 F 1 "+3V3" H 3915 5773 50  0000 C CNN
 F 2 "" H 3900 5600 50  0001 C CNN
@@
 F 0 "R1101" H 3968 1596 50  0000 L CNN
 F 1 "10k" H 3968 1505 50  0000 L CNN
-F 2 "" V 3940 1540 50  0001 C CNN
+F 2 "Resistor_SMD:R_0603_1608Metric_Pad1.05x0.95mm_HandSolder" V 3940 1540 50  0001 C CNN
 F 3 "~" H 3900 1550 50  0001 C CNN
-F 4 "" H 3900 1550 50  0001 C CNN "Digi-Key Link"
-F 5 "-" H 3900 1550 50  0001 C CNN "Digi-Key PN"
+F 4 "https://www.digikey.com/en/products/detail/yageo/RC0603FR-0710KL/726880?s=N4IgTCBcDaIEoGEAMA2JBmAYnAtEg7AIxIDSAMiALoC%2BQA" H 3900 1550 50  0001 C CNN "Digi-Key Link"
+F 5 "311-10.0KHRCT-ND" H 3900 1550 50  0001 C CNN "Digi-Key PN"
 	1    3900 1550
 	1    0    0    -1
@@
 P 5100 2450
 AR Path="/5F3FD151/5F8483D9" Ref="#PWR?"  Part="1"
-AR Path="/5F3FD151/5F82FB20/5F8483D9" Ref="#PWR01103"  Part="1"
-F 0 "#PWR01103" H 5100 2200 50  0001 C CNN
+AR Path="/5F3FD151/5F82FB20/5F8483D9" Ref="#PWR01107"  Part="1"
+F 0 "#PWR01107" H 5100 2200 50  0001 C CNN
 F 1 "GND" H 5105 2277 50  0000 C CNN
 F 2 "" H 5100 2450 50  0001 C CNN
@@
 F 0 "C1101" H 4215 2196 50  0000 L CNN
 F 1 "0.1uF" H 4215 2105 50  0000 L CNN
-F 2 "" H 4138 2000 50  0001 C CNN
+F 2 "Resistor_SMD:R_0603_1608Metric_Pad1.05x0.95mm_HandSolder" H 4138 2000 50  0001 C CNN
 F 3 "~" H 4100 2150 50  0001 C CNN
-F 4 "" H 4100 2150 50  0001 C CNN "Digi-Key Link"
-F 5 "-" H 4100 2150 50  0001 C CNN "Digi-Key PN"
+F 4 "https://www.digikey.com/en/products/detail/samsung-electro-mechanics/CL10B104KA8NNNC/3886664" H 4100 2150 50  0001 C CNN "Digi-Key Link"
+F 5 "1276-1006-1-ND" H 4100 2150 50  0001 C CNN "Digi-Key PN"
 	1    4100 2150
 	1    0    0    -1
@@
 P 4100 2450
 AR Path="/5F3FD151/5F8483F1" Ref="#PWR?"  Part="1"
-AR Path="/5F3FD151/5F82FB20/5F8483F1" Ref="#PWR01102"  Part="1"
-F 0 "#PWR01102" H 4100 2200 50  0001 C CNN
+AR Path="/5F3FD151/5F82FB20/5F8483F1" Ref="#PWR01104"  Part="1"
+F 0 "#PWR01104" H 4100 2200 50  0001 C CNN
 F 1 "GND" H 4105 2277 50  0000 C CNN
 F 2 "" H 4100 2450 50  0001 C CNN
@@
 P 5100 2200
 AR Path="/5F3FD151/5F8483FE" Ref="R?"  Part="1"
-AR Path="/5F3FD151/5F82FB20/5F8483FE" Ref="R1102"  Part="1"
-F 0 "R1102" H 5168 2246 50  0000 L CNN
+AR Path="/5F3FD151/5F82FB20/5F8483FE" Ref="R1104"  Part="1"
+F 0 "R1104" H 5168 2246 50  0000 L CNN
 F 1 "1k" H 5168 2155 50  0000 L CNN
-F 2 "" V 5140 2190 50  0001 C CNN
+F 2 "Resistor_SMD:R_0603_1608Metric_Pad1.05x0.95mm_HandSolder" V 5140 2190 50  0001 C CNN
 F 3 "~" H 5100 2200 50  0001 C CNN
-F 4 "" H 5100 2200 50  0001 C CNN "Digi-Key Link"
-F 5 "-" H 5100 2200 50  0001 C CNN "Digi-Key PN"
+F 4 "https://www.digikey.com/en/products/detail/yageo/RC0603FR-071KL/726843" H 5100 2200 50  0001 C CNN "Digi-Key Link"
+F 5 "311-1.00KHRCT-ND" H 5100 2200 50  0001 C CNN "Digi-Key PN"
 	1    5100 2200
 	1    0    0    -1
