File: Board Files/Breadboard_DMM/MCU.sch (KiCad schematic (older format))
At the start: 36 parts, among them J801 Conn_01x06, J802 AudioJack3, J803 Conn_02x02_Top_Bottom, Q801 NTZD3154N, SW801 SW_Push, SW802 SW_Push, SW803 SW_Push, SW804 SW_Push, SW805 SW_Push, U801 SI8422, U802 LCD-Generic_3.2in_SPI_SD, U803 STM32G030Kx

Commit message: Updated probe connector arrangement
Connections:
- net GNDL: now also J802.S; no longer J802.T
- net at U801.7 (B1): now also J802.T; no longer J802.S
Other:
- note removed: "MCU & Display"
- moved on the sheet: J802
Changed lines of the file:
@@
 Sheet 7 8
 Title "Toast-O-Meter"
-Date "2020-08-14"
+Date "2020-10-06"
 Rev "0"
 Comp ""
-Comment1 ""
+Comment1 "Isaac Rex"
 Comment2 ""
 Comment3 ""
@@
 U 1 1 5FBDEBF7
 P 3950 2650
-F 0 "J802" H 4050 2850 50  0000 R CNN
+F 0 "J802" H 4050 2400 50  0000 R CNN
 F 1 "AudioJack3" H 3670 2584 50  0001 R CNN
 F 2 "irex_Connector_Audio:Jack_3.5mm_CUI_SJ1-3523N_Horizontal" H 3950 2650 50  0001 C CNN
@@
 F 5 "CP1-3523N-ND" H 3950 2650 50  0001 C CNN "Digi-Key PN"
 	1    3950 2650
-	-1   0    0    -1
+	-1   0    0    1
 $EndComp
 $Comp
@@
 Wire Notes Line
 	10050 475  10050 3700
-Text Notes 12350 9725 0    200  ~ 40
-MCU & Display
 Text Notes 8950 4050 0    118  ~ 24
 Buttons
@@
 Wire Wire Line
 	12050 2100 12050 1925
-Wire Notes Line
-	12275 9275 12275 3700
 Text Label 13500 6400 0    50   ~ 0
 LCD_~RESET~
@@
 Wire Notes Line
 	13050 950  13050 3500
+Wire Notes Line
+	12350 9500 12350 3700
 $EndSCHEMATC

Commit message: Semi-finished component placement
Parts:
- added LS701: PKM13EPYH4000-A0, irex_Buzzer_Beeper:Buzzer_Murata_PKM13EPYH4000-A0_D12.6mm_H6.9mm, symbol Device:Speaker_Crystal
- added R707: 1k, Resistor_SMD:R_0603_1608Metric_Pad1.05x0.95mm_HandSolder, symbol Device:R_US
- added TP701, TP702: TestPoint, TestPoint:TestPoint_THTPad_D2.5mm_Drill1.2mm, symbol Connector:TestPoint
- C701: renamed from C801; footprint Resistor_SMD:R_0603_1608Metric_Pad1.05x0.95mm_HandSolder -> Capacitor_SMD:C_0603_1608Metric_Pad1.08x0.95mm_HandSolder
- C702: renamed from C802; footprint Resistor_SMD:R_0603_1608Metric_Pad1.05x0.95mm_HandSolder -> Capacitor_SMD:C_0603_1608Metric_Pad1.08x0.95mm_HandSolder
- C703: renamed from C803; footprint Resistor_SMD:R_0603_1608Metric_Pad1.05x0.95mm_HandSolder -> Capacitor_SMD:C_0603_1608Metric_Pad1.08x0.95mm_HandSolder
- C704: renamed from C804; footprint Resistor_SMD:R_0805_2012Metric_Pad1.15x1.40mm_HandSolder -> Capacitor_SMD:C_0805_2012Metric_Pad1.18x1.45mm_HandSolder
- C705: renamed from C805; footprint Resistor_SMD:R_0603_1608Metric_Pad1.05x0.95mm_HandSolder -> Capacitor_SMD:C_0603_1608Metric_Pad1.08x0.95mm_HandSolder
- C706: renamed from C806; footprint Resistor_SMD:R_0603_1608Metric_Pad1.05x0.95mm_HandSolder -> Capacitor_SMD:C_0603_1608Metric_Pad1.08x0.95mm_HandSolder
- C707: renamed from C807; footprint Resistor_SMD:R_0603_1608Metric_Pad1.05x0.95mm_HandSolder -> Capacitor_SMD:C_0603_1608Metric_Pad1.08x0.95mm_HandSolder
- C708: renamed from C808; footprint Resistor_SMD:R_0603_1608Metric_Pad1.05x0.95mm_HandSolder -> Capacitor_SMD:C_0603_1608Metric_Pad1.08x0.95mm_HandSolder
- D701: renamed from D801; symbol Device:D_ALT -> Device:D_Filled
- D702: renamed from D802; symbol Device:D_ALT -> Device:D_Filled
- J701: renamed from J801; footprint Connector_PinHeader_2.54mm:PinHeader_1x06_P2.54mm_Vertical -> Connector_PinHeader_2.54mm:PinHeader_1x06_P2.54mm_Horizontal; Digi-Key Link https://www.digikey.com/en/products/detail/adam-tech/PH1-06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 -> https://www.digikey.com/en/products/detail/adam-tech/ph1ra-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; Digi-Key PN 2057-PH1-06-UA-ND -> 2057-PH1RA-06-UA-ND
- J703: renamed from J803; footprint Connector_PinHeader_2.54mm:PinHeader_2x02_P2.54mm_Vertical -> Connector_PinHeader_2.54mm:PinHeader_2x02_P2.54mm_Horizontal; Digi-Key Link https://www.digikey.com/en/products/detail/adam-tech/PH2-04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 -> https://www.digikey.com/en/products/detail/adam-tech/PH2RA-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; Digi-Key PN 2057-PH2-04-UA-ND -> 2057-PH2RA-04-UA-ND
- Q701: renamed from Q801; value NTZD3154N -> BSD840N; footprint Package_TO_SOT_SMD:SOT-563 -> Package_TO_SOT_SMD:SOT-363_SC-70-6_Handsoldering; Digi-Key Link https://www.digikey.com/en/products/detail/on-semiconductor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 -> https://www.digikey.com/en/products/detail/infineon-technol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; Digi-Key PN NTZD3154NT1GOSCT-ND -> BSD840NH6327XTSA1CT-ND; MPN (none) -> BSD840NH6327XTSA1
- R703: renamed from R803; BOM (none) -> DNU
- SW701: renamed from SW801; BOM (none) -> DNU
- SW704: renamed from SW804; BOM (none) -> DNU
- U702: renamed from U802; symbol irex_Display_Graphic:LCD-Generic_3.2in_SPI_SD -> Breadboard_DMM-rescue:LCD-Generic_3.2in_SPI_SD-irex_Display_Graphic
- renumbered J802 to J702, R801 to R701, R802 to R702, R804 to R704, R805 to R705, R806 to R706, R807 to R708, R808 to R709, R809 to R710, R810 to R711, R811 to R712, R812 to R713, R813 to R714, R814 to R715, SW802 to SW702, SW803 to SW703, SW805 to SW705, U801 to U701, U803 to U703
Connections:
- net GND: now also LS701.2
- net at U703.2 (PC14): now also TP701.1
- net BUZZER: now reaches U703.20 (PC6)
- net BUZZER: now also R707.1
- net at U703.3 (PC15): now also TP702.1
- new net: LS701.1, R707.2
- no-connect marks 4 -> 1
Other:
- note added: "Buzzer"
- moved on the sheet: C704, C705, C707, R712, SW704, U703
