File: Board Files/Breadboard_DMM/MCU.sch (KiCad schematic (older format))
At the start: 40 parts, among them J701 Conn_01x06, J702 AudioJack3, J703 Conn_02x02_Top_Bottom, Q701 BSD840N, SW701 SW_Push, SW702 SW_Push, SW703 SW_Push, SW704 SW_Push, SW705 SW_Push, U701 SI8422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

Commit message: 59 unrouted nodes
Parts:
- TP701, TP702: footprint TestPoint:TestPoint_THTPad_D2.5mm_Drill1.2mm -> TestPoint:TestPoint_THTPad_D1.5mm_Drill0.7mm
Connections:
- net ADC_~DRDY: now also U703.7 (PA0); no longer U703.8 (PA1)
- net VREF_4.096V_~EN: now also U703.8 (PA1); no longer U703.7 (PA0)
Changed lines of the file:
@@
 Text HLabel 3750 7750 0    50   Output ~ 0
 CALIBRATE_MUX_~A
-Text HLabel 6300 6850 2    50   Output ~ 0
+Text HLabel 6300 6950 2    50   Output ~ 0
 VREF_4.096V_~EN
 Wire Wire Line
 	6300 6850 5450 6850
-Text HLabel 6300 6950 2    50   Input ~ 0
+Text HLabel 6300 6850 2    50   Input ~ 0
 ADC_~DRDY
 Wire Wire Line
@@
 U 1 1 5F94BDCF
 P 4000 7150
-F 0 "TP701" V 4000 7400 50  0000 C CNN
+F 0 "TP701" V 4000 7450 50  0000 C CNN
 F 1 "TestPoint" V 4104 7222 50  0001 C CNN
-F 2 "TestPoint:TestPoint_THTPad_D2.5mm_Drill1.2mm" H 4200 7150 50  0001 C CNN
+F 2 "TestPoint:TestPoint_THTPad_D1.5mm_Drill0.7mm" H 4200 7150 50  0001 C CNN
 F 3 "~" H 4200 7150 50  0001 C CNN
 F 4 "2057-PH2-10-UA-ND" H 4000 7150 50  0001 C CNN "Digi-Key PN"
@@
 U 1 1 5F94C0A7
 P 4000 7250
-F 0 "TP702" V 4000 7500 50  0000 C CNN
+F 0 "TP702" V 4000 7550 50  0000 C CNN
 F 1 "TestPoint" V 4104 7322 50  0001 C CNN
-F 2 "TestPoint:TestPoint_THTPad_D2.5mm_Drill1.2mm" H 4200 7250 50  0001 C CNN
+F 2 "TestPoint:TestPoint_THTPad_D1.5mm_Drill0.7mm" H 4200 7250 50  0001 C CNN
 F 3 "~" H 4200 7250 50  0001 C CNN
 F 4 "2057-PH2-10-UA-ND" H 4000 7250 50  0001 C CNN "Digi-Key PN"

Commit message: Added silkscreen graphics and BOM
Parts:
- DS701: renamed from U702; footprint irex_Display:LCD-Generic-3.2in_89.30x55.04mm -> irex_Display:LCD-Generic-3.2in_89.30x55.04mm_ReducedCourtyard; symbol Breadboard_DMM-rescue:LCD-Generic_3.2in_SPI_SD-irex_Display_Graphic -> irex_Display_Graphic:LCD-Generic_3.2in_SPI_SD
- R707: Digi-Key Link https://www.digikey.com/en/products/detail/yageo/RC0603FR-07100RL/726888 -> https://www.digikey.com/en/products/detail/yageo/RC0603FR-071KL/726843; Digi-Key PN 311-100HRCT-ND -> 311-1.00KHRCT-ND
- renumbered U703 to U702
Changed lines of the file:
@@
 	4850 6550 4850 5400
 $Comp
-L irex_MCU_ST_STM32G0:STM32G030Kx U703
+L irex_MCU_ST_STM32G0:STM32G030Kx U702
 U 1 1 5F3FD47F
 P 4850 7550
-F 0 "U703" H 4350 8600 50  0000 L CNN
+F 0 "U702" H 4350 8600 50  0000 L CNN
 F 1 "STM32G030Kx" H 4500 8500 50  0000 C CNN
 F 2 "Package_QFP:LQFP-32_7x7mm_P0.8mm" H 5700 6500 50  0001 C CNN
@@
 Display
 $Comp
-L Breadboard_DMM-rescue:LCD-Generic_3.2in_SPI_SD-irex_Display_Graphic U?
+L irex_Display_Graphic:LCD-Generic_3.2in_SPI_SD DS?
 U 1 1 5F4ADAFA
 P 14500 6800
-AR Path="/5F4ADAFA" Ref="U?"  Part="1"
-AR Path="/5F3FD151/5F4ADAFA" Ref="U702"  Part="1"
-F 0 "U702" H 14100 7650 50  0000 L CNN
+AR Path="/5F4ADAFA" Ref="DS?"  Part="1"
+AR Path="/5F3FD151/5F4ADAFA" Ref="DS701"  Part="1"
+F 0 "DS701" H 14100 7650 50  0000 L CNN
 F 1 "LCD-Generic_3.2in_SPI_SD" H 14400 7550 50  0000 R CNN
-F 2 "irex_Display:LCD-Generic-3.2in_89.30x55.04mm" H 15500 6000 50  0001 C CNN
+F 2 "irex_Display:LCD-Generic-3.2in_89.30x55.04mm_ReducedCourtyard" H 15500 6000 50  0001 C CNN
 F 3 "https://www.aliexpress.com/item/4001122632293.html?spm=a2g0o.productlist.0.0.626763a37DWpAR&algo_pvid=075ffa5b-9e24-45ec-b277-c66fde4fd636&algo_expid=075ffa5b-9e24-45ec-b277-c66fde4fd636-8&btsid=0be3746c15983696518323585e6542&ws_ab_test=searchweb0_0,searchweb201602_,searchweb201603_" H 14400 7200 50  0001 C CNN
 F 4 "https://www.digikey.com/en/products/detail/samtec-inc/SLW-104-01-T-S/1104832 ; https://www.digikey.com/en/products/detail/samtec-inc/SLW-114-01-T-S/1104822" H 14500 6800 50  0001 C CNN "Digi-Key Link"
@@
 F 2 "Resistor_SMD:R_0603_1608Metric_Pad1.05x0.95mm_HandSolder" V 14290 4240 50  0001 C CNN
 F 3 "~" H 14250 4250 50  0001 C CNN
-F 4 "https://www.digikey.com/en/products/detail/yageo/RC0603FR-07100RL/726888" H 14250 4250 50  0001 C CNN "Digi-Key Link"
-F 5 "311-100HRCT-ND" H 14250 4250 50  0001 C CNN "Digi-Key PN"
+F 4 "https://www.digikey.com/en/products/detail/yageo/RC0603FR-071KL/726843" H 14250 4250 50  0001 C CNN "Digi-Key Link"
+F 5 "311-1.00KHRCT-ND" H 14250 4250 50  0001 C CNN "Digi-Key PN"
 	1    14250 4250
 	0    -1   -1   0
