File: Board Files/Breadboard_DMM/Ohmeter Current Source.sch (KiCad schematic (older format))
At the start: 20 parts, among them Q501 NTZD3154N, Q502 NTZD3154N, U501 LMV358, U502 MCP1501

Commit message: Semi-finished component placement
Parts:
- C401: renamed from C501; footprint Resistor_SMD:R_0603_1608Metric_Pad1.05x0.95mm_HandSolder -> Capacitor_SMD:C_0603_1608Metric_Pad1.08x0.95mm_HandSolder
- C402: renamed from C502; footprint Resistor_SMD:R_0603_1608Metric_Pad1.05x0.95mm_HandSolder -> Capacitor_SMD:C_0603_1608Metric_Pad1.08x0.95mm_HandSolder
- C403: renamed from C503; footprint Resistor_SMD:R_0603_1608Metric_Pad1.05x0.95mm_HandSolder -> Capacitor_SMD:C_0603_1608Metric_Pad1.08x0.95mm_HandSolder
- D401: renamed from D501; symbol Device:D_TVS_ALT -> Device:D_TVS_Filled
- Q401: renamed from Q501; value NTZD3154N -> BSD840N; footprint Package_TO_SOT_SMD:SOT-563 -> Package_TO_SOT_SMD:SOT-363_SC-70-6_Handsoldering; Digi-Key Link https://www.digikey.com/en/products/detail/on-semiconductor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 -> https://www.digikey.com/en/products/detail/infineon-technol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; Digi-Key PN NTZD3154NT1GOSCT-ND -> BSD840NH6327XTSA1CT-ND; MPN (none) -> BSD840NH6327XTSA1
- Q402: renamed from Q502; value NTZD3154N -> BSD840N; footprint Package_TO_SOT_SMD:SOT-563 -> Package_TO_SOT_SMD:SOT-363_SC-70-6_Handsoldering; Digi-Key Link https://www.digikey.com/en/products/detail/on-semiconductor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 -> https://www.digikey.com/en/products/detail/infineon-technol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; Digi-Key PN NTZD3154NT1GOSCT-ND -> BSD840NH6327XTSA1CT-ND; MPN (none) -> BSD840NH6327XTSA1
- R402: renamed from R502; value 10k -> 1k; Digi-Key Link https://www.digikey.com/en/products/detail/yageo/RC0603FR-0710KL/726880?s=N4IgTCBcDaIEoGEAMA2JBmAYnAtEg7AIxIDSAMiALoC%2BQA -> https://www.digikey.com/en/products/detail/yageo/RC0603FR-071KL/726843; Digi-Key PN 311-10.0KHRCT-ND -> 311-1.00KHRCT-ND
- renumbered R501 to R401, R503 to R403, R504 to R404, R505 to R405, R506 to R406, R507 to R407, R508 to R408, R509 to R409, R510 to R410, R511 to R411, R512 to R412, U501 to U401, U502 to U402
Other:
- note added: "TODO: Consider MAX6071AAUT12+T \nas current source"
- moved on the sheet: Q401A, Q401B
