File: Board Files/Breadboard_DMM/Power_Input_Protection.sch (KiCad schematic (older format))
At the start: 10 parts

Commit message: Finished main cleanup, started adding digikey part numbers
Parts:
- Q301: renamed from Q?; Digi-Key Link (none) -> https://www.digikey.com/en/products/detail/diodes-incorpora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; Digi-Key PN (none) -> DMP3085LSD-13DICT-ND; MPN (none) -> DMP3085LSD
- Q302: renamed from Q?; Digi-Key Link (none) -> https://www.digikey.com/en/products/detail/nexperia-usa-inc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; Digi-Key PN (none) -> 1727-2958-1-ND
- R301, R302, R303, R304, R305, R306: renamed from R?; Digi-Key PN (none) -> -
- U301: renamed from U?; Digi-Key Link (none) -> https://www.digikey.com/en/products/detail/texas-instrument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; Digi-Key PN (none) -> 296-53244-1-ND; MPN (none) -> TL432LI
Changed lines of the file:
@@
 $Descr A4 11693 8268
 encoding utf-8
-Sheet 9 9
+Sheet 3 10
 Title "Toast-O-Meter"
 Date ""
@@
 P 4000 3250
 AR Path="/5FDFAE85/5F7D131D" Ref="R?"  Part="1"
-AR Path="/5F7CCAA0/5F7D131D" Ref="R?"  Part="1"
-F 0 "R?" H 3932 3204 50  0000 R CNN
+AR Path="/5F7CCAA0/5F7D131D" Ref="R304"  Part="1"
+F 0 "R304" H 3932 3204 50  0000 R CNN
 F 1 "10k" H 3932 3295 50  0000 R CNN
 F 2 "" V 4040 3240 50  0001 C CNN
 F 3 "~" H 4000 3250 50  0001 C CNN
+F 4 "" H 4000 3250 50  0001 C CNN "Digi-Key Link"
+F 5 "-" H 4000 3250 50  0001 C CNN "Digi-Key PN"
 	1    4000 3250
 	-1   0    0    1
@@
 P 6000 3000
 AR Path="/5FDFAE85/5F7D1D7F" Ref="R?"  Part="1"
-AR Path="/5F7CCAA0/5F7D1D7F" Ref="R?"  Part="1"
-F 0 "R?" V 5800 2950 50  0000 L CNN
+AR Path="/5F7CCAA0/5F7D1D7F" Ref="R302"  Part="1"
+F 0 "R302" V 5800 2950 50  0000 L CNN
 F 1 "10k" V 5900 2950 50  0000 L CNN
 F 2 "" V 6040 2990 50  0001 C CNN
 F 3 "~" H 6000 3000 50  0001 C CNN
+F 4 "" H 6000 3000 50  0001 C CNN "Digi-Key Link"
+F 5 "-" H 6000 3000 50  0001 C CNN "Digi-Key PN"
 	1    6000 3000
 	0    1    1    0
@@
 P 7250 3600
 AR Path="/5FDFAE85/5F7D260A" Ref="R?"  Part="1"
-AR Path="/5F7CCAA0/5F7D260A" Ref="R?"  Part="1"
-F 0 "R?" H 7182 3554 50  0000 R CNN
+AR Path="/5F7CCAA0/5F7D260A" Ref="R305"  Part="1"
+F 0 "R305" H 7182 3554 50  0000 R CNN
 F 1 "10k" H 7182 3645 50  0000 R CNN
 F 2 "" V 7290 3590 50  0001 C CNN
 F 3 "~" H 7250 3600 50  0001 C CNN
+F 4 "" H 7250 3600 50  0001 C CNN "Digi-Key Link"
+F 5 "-" H 7250 3600 50  0001 C CNN "Digi-Key PN"
 	1    7250 3600
 	-1   0    0    1
 $EndComp
 $Comp
-L irex_Transistor_FET:DMP3085LSD Q?
+L irex_Transistor_FET:DMP3085LSD Q301
 U 1 1 5F7DB1F5
 P 4000 2600
-F 0 "Q?" V 4425 2600 50  0000 C CNN
+F 0 "Q301" V 4425 2600 50  0000 C CNN
 F 1 "DMP3085LSD" V 4334 2600 50  0000 C CNN
 F 2 "Package_SO:SO-8_3.9x4.9mm_P1.27mm" H 4200 2450 50  0001 L CNN
 F 3 "https://www.diodes.com/assets/Datasheets/DMP3085LSD.pdf" H 4050 2600 50  0001 C CNN
+F 4 "https://www.digikey.com/en/products/detail/diodes-incorporated/DMP3085LSD-13/4251594" H 4000 2600 50  0001 C CNN "Digi-Key Link"
+F 5 "DMP3085LSD-13DICT-ND" H 4000 2600 50  0001 C CNN "Digi-Key PN"
+F 6 "DMP3085LSD" H 4000 2600 50  0001 C CNN "MPN"
 	1    4000 2600
 	0    -1   -1   0
 $EndComp
 $Comp
-L irex_Transistor_FET:DMP3085LSD Q?
+L irex_Transistor_FET:DMP3085LSD Q301
 U 2 1 5F7DDE08
 P 7250 2600
-F 0 "Q?" V 7675 2600 50  0000 C CNN
+F 0 "Q301" V 7675 2600 50  0000 C CNN
 F 1 "DMP3085LSD" V 7584 2600 50  0000 C CNN
 F 2 "Package_SO:SO-8_3.9x4.9mm_P1.27mm" H 7450 2450 50  0001 L CNN
 F 3 "https://www.diodes.com/assets/Datasheets/DMP3085LSD.pdf" H 7300 2600 50  0001 C CNN
+F 4 "https://www.digikey.com/en/products/detail/diodes-incorporated/DMP3085LSD-13/4251594" H 7250 2600 50  0001 C CNN "Digi-Key Link"
+F 5 "DMP3085LSD-13DICT-ND" H 7250 2600 50  0001 C CNN "Digi-Key PN"
+F 6 "DMP3085LSD" H 7250 2600 50  0001 C CNN "MPN"
 	2    7250 2600
 	0    1    -1   0
@@
 P 5550 2750
 AR Path="/5FDFAE85/5F7E105A" Ref="R?"  Part="1"
-AR Path="/5F7CCAA0/5F7E105A" Ref="R?"  Part="1"
-F 0 "R?" H 5482 2704 50  0000 R CNN
+AR Path="/5F7CCAA0/5F7E105A" Ref="R301"  Part="1"
+F 0 "R301" H 5482 2704 50  0000 R CNN
 F 1 "1.5k" H 5482 2795 50  0000 R CNN
 F 2 "" V 5590 2740 50  0001 C CNN
 F 3 "~" H 5550 2750 50  0001 C CNN
+F 4 "" H 5550 2750 50  0001 C CNN "Digi-Key Link"
+F 5 "-" H 5550 2750 50  0001 C CNN "Digi-Key PN"
 	1    5550 2750
 	-1   0    0    1
@@
 	5150 3350 5450 3350
 $Comp
-L irex_Reference_Voltage:TL432LI U?
+L irex_Reference_Voltage:TL432LI U301
 U 1 1 5F7E207E
 P 5550 3350
-F 0 "U?" V 5596 3280 50  0000 R CNN
+F 0 "U301" V 5596 3280 50  0000 R CNN
 F 1 "TL432LI" V 5505 3280 50  0000 R CNN
 F 2 "Package_TO_SOT_SMD:SOT-23" H 5550 3200 50  0001 C CIN
 F 3 "https://www.ti.com/lit/ds/symlink/tl431li.pdf?HQS=TI-null-null-digikeymode-df-pf-null-wwe&ts=1601074554367" H 5550 3350 50  0001 C CIN
+F 4 "https://www.digikey.com/en/products/detail/texas-instruments/TL432LIACDBZR/9860322" H 5550 3350 50  0001 C CNN "Digi-Key Link"
+F 5 "296-53244-1-ND" H 5550 3350 50  0001 C CNN "Digi-Key PN"
+F 6 "TL432LI" H 5550 3350 50  0001 C CNN "MPN"
 	1    5550 3350
 	0    -1   -1   0
@@
 P 5150 3650
 AR Path="/5FDFAE85/5F7D15E1" Ref="R?"  Part="1"
-AR Path="/5F7CCAA0/5F7D15E1" Ref="R?"  Part="1"
-F 0 "R?" H 5082 3604 50  0000 R CNN
+AR Path="/5F7CCAA0/5F7D15E1" Ref="R306"  Part="1"
+F 0 "R306" H 5082 3604 50  0000 R CNN
 F 1 "10k" H 5082 3695 50  0000 R CNN
 F 2 "" V 5190 3640 50  0001 C CNN
 F 3 "~" H 5150 3650 50  0001 C CNN
+F 4 "" H 5150 3650 50  0001 C CNN "Digi-Key Link"
+F 5 "-" H 5150 3650 50  0001 C CNN "Digi-Key PN"
 	1    5150 3650
 	-1   0    0    1
@@
 P 5150 3050
 AR Path="/5FDFAE85/5F7E0D9C" Ref="R?"  Part="1"
-AR Path="/5F7CCAA0/5F7E0D9C" Ref="R?"  Part="1"
-F 0 "R?" H 5082 3004 50  0000 R CNN
+AR Path="/5F7CCAA0/5F7E0D9C" Ref="R303"  Part="1"
+F 0 "R303" H 5082 3004 50  0000 R CNN
 F 1 "12k" H 5082 3095 50  0000 R CNN
 F 2 "" V 5190 3040 50  0001 C CNN
 F 3 "~" H 5150 3050 50  0001 C CNN
+F 4 "" H 5150 3050 50  0001 C CNN "Digi-Key Link"
+F 5 "-" H 5150 3050 50  0001 C CNN "Digi-Key PN"
 	1    5150 3050
 	-1   0    0    1
@@
 	7250 2800 7250 3300
 $Comp
-L Device:Q_PNP_BEC Q?
+L Device:Q_PNP_BEC Q302
 U 1 1 5F81D169
 P 6550 3000
-F 0 "Q?" H 6741 3046 50  0000 L CNN
+F 0 "Q302" H 6741 3046 50  0000 L CNN
 F 1 "PMBT2907A" H 6741 2955 50  0000 L CNN
 F 2 "Package_TO_SOT_SMD:SOT-23_Handsoldering" H 6750 3100 50  0001 C CNN
 F 3 "https://media.digikey.com/pdf/Data%20Sheets/NXP%20PDFs/PMBT2907(A).pdf" H 6550 3000 50  0001 C CNN
 F 4 "PMBT2907A" H 6550 3000 50  0001 C CNN "MPN"
+F 5 "https://www.digikey.com/en/products/detail/nexperia-usa-inc/PMBT2907A215/763344" H 6550 3000 50  0001 C CNN "Digi-Key Link"
+F 6 "1727-2958-1-ND" H 6550 3000 50  0001 C CNN "Digi-Key PN"
 	1    6550 3000
 	1    0    0    -1

Commit message: Finished adding parts, cleaned up, ran ERC
Parts:
- R301: footprint (none) -> Resistor_SMD:R_0603_1608Metric_Pad1.05x0.95mm_HandSolder; Digi-Key Link (none) -> https://www.digikey.com/en/products/detail/yageo/RC0603FR-0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; Digi-Key PN - -> 311-1.50KHRCT-ND
- R302, R304, R305, R306: footprint (none) -> Resistor_SMD:R_0603_1608Metric_Pad1.05x0.95mm_HandSolder; Digi-Key Link (none) -> https://www.digikey.com/en/products/detail/yageo/RC0603FR-0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; Digi-Key PN - -> 311-10.0KHRCT-ND
- R303: footprint (none) -> Resistor_SMD:R_0603_1608Metric_Pad1.05x0.95mm_HandSolder; Digi-Key Link (none) -> https://www.digikey.com/en/products/detail/yageo/RC0603FR-0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; Digi-Key PN - -> 311-12.0KHRCT-ND
Other:
- note added: "Vin Protection"
- moved on the sheet: Q301A, Q301B, Q302, R?, U301

Commit message: Cleaned up files
Other:
- note added: "Power Input Protection"
- note removed: "Vin Protection"
Changed lines of the file:
@@
 $Descr USLedger 17000 11000
 encoding utf-8
-Sheet 3 8
+Sheet 8 8
 Title "Toast-O-Meter"
 Date "2020-08-14"
@@
 AR Path="/5F7CCAA0/5F7D131D" Ref="R304"  Part="1"
 AR Path="/602C5383/5F7D131D" Ref="R?"  Part="1"
-F 0 "R?" H 6182 5554 50  0000 R CNN
+F 0 "R304" H 6182 5554 50  0000 R CNN
 F 1 "10k" H 6182 5645 50  0000 R CNN
 F 2 "Resistor_SMD:R_0603_1608Metric_Pad1.05x0.95mm_HandSolder" V 6290 5590 50  0001 C CNN
@@
 AR Path="/5F7CCAA0/5F7D1D7F" Ref="R302"  Part="1"
 AR Path="/602C5383/5F7D1D7F" Ref="R?"  Part="1"
-F 0 "R?" V 9200 5200 50  0000 L CNN
+F 0 "R302" V 9200 5200 50  0000 L CNN
 F 1 "10k" V 9300 5200 50  0000 L CNN
 F 2 "Resistor_SMD:R_0603_1608Metric_Pad1.05x0.95mm_HandSolder" V 9440 5240 50  0001 C CNN
@@
 AR Path="/5F7CCAA0/5F7D260A" Ref="R305"  Part="1"
 AR Path="/602C5383/5F7D260A" Ref="R?"  Part="1"
-F 0 "R?" H 10582 5904 50  0000 R CNN
+F 0 "R305" H 10582 5904 50  0000 R CNN
 F 1 "10k" H 10582 5995 50  0000 R CNN
 F 2 "Resistor_SMD:R_0603_1608Metric_Pad1.05x0.95mm_HandSolder" V 10690 5940 50  0001 C CNN
@@
 AR Path="/5F7CCAA0/5F7DB1F5" Ref="Q301"  Part="1"
 AR Path="/602C5383/5F7DB1F5" Ref="Q?"  Part="1"
-F 0 "Q?" V 6675 4700 50  0000 C CNN
+F 0 "Q301" V 6675 4700 50  0000 C CNN
 F 1 "DMP3085LSD" V 6584 4700 50  0000 C CNN
 F 2 "Package_SO:SO-8_3.9x4.9mm_P1.27mm" H 6450 4550 50  0001 L CNN
@@
 AR Path="/5F7CCAA0/5F7DDE08" Ref="Q301"  Part="2"
 AR Path="/602C5383/5F7DDE08" Ref="Q?"  Part="2"
-F 0 "Q?" V 11075 4700 50  0000 C CNN
+F 0 "Q301" V 11075 4700 50  0000 C CNN
 F 1 "DMP3085LSD" V 10984 4700 50  0000 C CNN
 F 2 "Package_SO:SO-8_3.9x4.9mm_P1.27mm" H 10850 4550 50  0001 L CNN
@@
 AR Path="/5F7CCAA0/5F7E105A" Ref="R301"  Part="1"
 AR Path="/602C5383/5F7E105A" Ref="R?"  Part="1"
-F 0 "R?" H 8882 4904 50  0000 R CNN
+F 0 "R301" H 8882 4904 50  0000 R CNN
 F 1 "1.5k" H 8882 4995 50  0000 R CNN
 F 2 "Resistor_SMD:R_0603_1608Metric_Pad1.05x0.95mm_HandSolder" V 8990 4940 50  0001 C CNN
@@
 AR Path="/5F7CCAA0/5F7E207E" Ref="U301"  Part="1"
 AR Path="/602C5383/5F7E207E" Ref="U?"  Part="1"
-F 0 "U?" V 8996 5630 50  0000 R CNN
+F 0 "U301" V 8996 5630 50  0000 R CNN
 F 1 "TL432LI" V 8905 5630 50  0000 R CNN
 F 2 "Package_TO_SOT_SMD:SOT-23" H 8950 5550 50  0001 C CIN
@@
 AR Path="/5F7CCAA0/5F7D15E1" Ref="R306"  Part="1"
 AR Path="/602C5383/5F7D15E1" Ref="R?"  Part="1"
-F 0 "R?" H 8282 6054 50  0000 R CNN
+F 0 "R306" H 8282 6054 50  0000 R CNN
 F 1 "10k" H 8282 6145 50  0000 R CNN
 F 2 "Resistor_SMD:R_0603_1608Metric_Pad1.05x0.95mm_HandSolder" V 8390 6090 50  0001 C CNN
@@
 AR Path="/5F7CCAA0/5F7E0D9C" Ref="R303"  Part="1"
 AR Path="/602C5383/5F7E0D9C" Ref="R?"  Part="1"
-F 0 "R?" H 8282 5254 50  0000 R CNN
+F 0 "R303" H 8282 5254 50  0000 R CNN
 F 1 "12k" H 8282 5345 50  0000 R CNN
 F 2 "Resistor_SMD:R_0603_1608Metric_Pad1.05x0.95mm_HandSolder" V 8390 5290 50  0001 C CNN
@@
 AR Path="/5F7CCAA0/5F81D169" Ref="Q302"  Part="1"
 AR Path="/602C5383/5F81D169" Ref="Q?"  Part="1"
-F 0 "Q?" H 10141 5296 50  0000 L CNN
+F 0 "Q302" H 10141 5296 50  0000 L CNN
 F 1 "PMBT2907A" H 10141 5205 50  0000 L CNN
 F 2 "Package_TO_SOT_SMD:SOT-23_Handsoldering" H 10150 5350 50  0001 C CNN
@@
 	10300 5950 10300 6300
 Text Notes 12400 9750 0    200  ~ 40
-Vin Protection
+Power Input Protection
 $EndSCHEMATC

Commit message: Updated probe connector arrangement
Other:
- note removed: "Power Input Protection"
Changed lines of the file:
@@
 Sheet 8 8
 Title "Toast-O-Meter"
-Date "2020-08-14"
+Date "2020-10-06"
 Rev "0"
 Comp ""
-Comment1 ""
+Comment1 "Isaac Rex"
 Comment2 ""
 Comment3 ""
@@
 Wire Notes Line style solid
 	10300 5950 10300 6300
-Text Notes 12400 9750 0    200  ~ 40
-Power Input Protection
 $EndSCHEMATC

Commit message: Semi-finished component placement
Parts:
- removed R304: 10k, Resistor_SMD:R_0603_1608Metric_Pad1.05x0.95mm_HandSolder, symbol Device:R_US
- renumbered Q301 to Q801, Q302 to Q802, R301 to R801, R302 to R802, R303 to R803, R305 to R804, R306 to R805, U301 to U801
Connections:
- net V_IN-: now also Q801.2 (G)
- net V_IN+_REV_PROTECTED: now reaches Q801.1 (S), Q801.3 (S), Q802.3 (C), R801.2, R803.2
Other:
- note added: "Acts as a comparator and\ngoes low when Vin = 5.5V.\nInternal Vref = 2.495V"
- note removed: "U? acts as a comparator and\ngoes low when Vin = 5.5V.\nInternal Vref = 2.495V"
Changed lines of the file:
@@
-$Comp
-L Device:R_US R?
-U 1 1 5F7D131D
-P 6250 5600
-AR Path="/5FDFAE85/5F7D131D" Ref="R?"  Part="1"
-AR Path="/5F7CCAA0/5F7D131D" Ref="R304"  Part="1"
-AR Path="/602C5383/5F7D131D" Ref="R?"  Part="1"
-F 0 "R304" H 6182 5554 50  0000 R CNN
-F 1 "10k" H 6182 5645 50  0000 R CNN
-F 2 "Resistor_SMD:R_0603_1608Metric_Pad1.05x0.95mm_HandSolder" V 6290 5590 50  0001 C CNN
-F 3 "~" H 6250 5600 50  0001 C CNN
-F 4 "https://www.digikey.com/en/products/detail/yageo/RC0603FR-0710KL/726880?s=N4IgTCBcDaIEoGEAMA2JBmAYnAtEg7AIxIDSAMiALoC%2BQA" H 6250 5600 50  0001 C CNN "Digi-Key Link"
-F 5 "311-10.0KHRCT-ND" H 6250 5600 50  0001 C CNN "Digi-Key PN"
-	1    6250 5600
-	-1   0    0    1
-$EndComp
 $Comp
 L Device:R_US R?
@@
 P 9400 5250
 AR Path="/5FDFAE85/5F7D1D7F" Ref="R?"  Part="1"
-AR Path="/5F7CCAA0/5F7D1D7F" Ref="R302"  Part="1"
+AR Path="/5F7CCAA0/5F7D1D7F" Ref="R802"  Part="1"
 AR Path="/602C5383/5F7D1D7F" Ref="R?"  Part="1"
-F 0 "R302" V 9200 5200 50  0000 L CNN
+F 0 "R802" V 9200 5200 50  0000 L CNN
 F 1 "10k" V 9300 5200 50  0000 L CNN
 F 2 "Resistor_SMD:R_0603_1608Metric_Pad1.05x0.95mm_HandSolder" V 9440 5240 50  0001 C CNN
@@
 P 10650 5950
 AR Path="/5FDFAE85/5F7D260A" Ref="R?"  Part="1"
-AR Path="/5F7CCAA0/5F7D260A" Ref="R305"  Part="1"
+AR Path="/5F7CCAA0/5F7D260A" Ref="R804"  Part="1"
 AR Path="/602C5383/5F7D260A" Ref="R?"  Part="1"
-F 0 "R305" H 10582 5904 50  0000 R CNN
+F 0 "R804" H 10582 5904 50  0000 R CNN
 F 1 "10k" H 10582 5995 50  0000 R CNN
 F 2 "Resistor_SMD:R_0603_1608Metric_Pad1.05x0.95mm_HandSolder" V 10690 5940 50  0001 C CNN
@@
 $EndComp
 $Comp
-L irex_Transistor_FET:DMP3085LSD Q301
+L irex_Transistor_FET:DMP3085LSD Q801
 U 1 1 5F7DB1F5
 P 6250 4700
-AR Path="/5F7CCAA0/5F7DB1F5" Ref="Q301"  Part="1"
+AR Path="/5F7CCAA0/5F7DB1F5" Ref="Q801"  Part="1"
 AR Path="/602C5383/5F7DB1F5" Ref="Q?"  Part="1"
-F 0 "Q301" V 6675 4700 50  0000 C CNN
+F 0 "Q801" V 6675 4700 50  0000 C CNN
 F 1 "DMP3085LSD" V 6584 4700 50  0000 C CNN
 F 2 "Package_SO:SO-8_3.9x4.9mm_P1.27mm" H 6450 4550 50  0001 L CNN
@@
 $EndComp
 $Comp
-L irex_Transistor_FET:DMP3085LSD Q301
+L irex_Transistor_FET:DMP3085LSD Q801
 U 2 1 5F7DDE08
 P 10650 4700
-AR Path="/5F7CCAA0/5F7DDE08" Ref="Q301"  Part="2"
+AR Path="/5F7CCAA0/5F7DDE08" Ref="Q801"  Part="2"
 AR Path="/602C5383/5F7DDE08" Ref="Q?"  Part="2"
-F 0 "Q301" V 11075 4700 50  0000 C CNN
+F 0 "Q801" V 11075 4700 50  0000 C CNN
 F 1 "DMP3085LSD" V 10984 4700 50  0000 C CNN
 F 2 "Package_SO:SO-8_3.9x4.9mm_P1.27mm" H 10850 4550 50  0001 L CNN
@@
 P 8950 4950
 AR Path="/5FDFAE85/5F7E105A" Ref="R?"  Part="1"
-AR Path="/5F7CCAA0/5F7E105A" Ref="R301"  Part="1"
+AR Path="/5F7CCAA0/5F7E105A" Ref="R801"  Part="1"
 AR Path="/602C5383/5F7E105A" Ref="R?"  Part="1"
-F 0 "R301" H 8882 4904 50  0000 R CNN
+F 0 "R801" H 8882 4904 50  0000 R CNN
 F 1 "1.5k" H 8882 4995 50  0000 R CNN
 F 2 "Resistor_SMD:R_0603_1608Metric_Pad1.05x0.95mm_HandSolder" V 8990 4940 50  0001 C CNN
@@
 $EndComp
 Wire Wire Line
-	6250 5450 6250 4900
-Wire Wire Line
 	8950 5100 8950 5250
 Wire Wire Line
@@
 Connection ~ 8350 5700
 Wire Wire Line
-	6250 5750 6250 6550
-Wire Wire Line
 	10650 6100 10650 6550
 Wire Wire Line
 	8350 5700 8850 5700
 $Comp
-L irex_Reference_Voltage:TL432LI U301
+L irex_Reference_Voltage:TL432LI U801
 U 1 1 5F7E207E
 P 8950 5700
-AR Path="/5F7CCAA0/5F7E207E" Ref="U301"  Part="1"
+AR Path="/5F7CCAA0/5F7E207E" Ref="U801"  Part="1"
 AR Path="/602C5383/5F7E207E" Ref="U?"  Part="1"
-F 0 "U301" V 8996 5630 50  0000 R CNN
+F 0 "U801" V 8996 5630 50  0000 R CNN
 F 1 "TL432LI" V 8905 5630 50  0000 R CNN
 F 2 "Package_TO_SOT_SMD:SOT-23" H 8950 5550 50  0001 C CIN
@@
 P 8350 6100
 AR Path="/5FDFAE85/5F7D15E1" Ref="R?"  Part="1"
-AR Path="/5F7CCAA0/5F7D15E1" Ref="R306"  Part="1"
+AR Path="/5F7CCAA0/5F7D15E1" Ref="R805"  Part="1"
 AR Path="/602C5383/5F7D15E1" Ref="R?"  Part="1"
-F 0 "R306" H 8282 6054 50  0000 R CNN
+F 0 "R805" H 8282 6054 50  0000 R CNN
 F 1 "10k" H 8282 6145 50  0000 R CNN
 F 2 "Resistor_SMD:R_0603_1608Metric_Pad1.05x0.95mm_HandSolder" V 8390 6090 50  0001 C CNN
@@
 P 8350 5300
 AR Path="/5FDFAE85/5F7E0D9C" Ref="R?"  Part="1"
-AR Path="/5F7CCAA0/5F7E0D9C" Ref="R303"  Part="1"
+AR Path="/5F7CCAA0/5F7E0D9C" Ref="R803"  Part="1"
 AR Path="/602C5383/5F7E0D9C" Ref="R?"  Part="1"
-F 0 "R303" H 8282 5254 50  0000 R CNN
+F 0 "R803" H 8282 5254 50  0000 R CNN
 F 1 "12k" H 8282 5345 50  0000 R CNN
 F 2 "Resistor_SMD:R_0603_1608Metric_Pad1.05x0.95mm_HandSolder" V 8390 5290 50  0001 C CNN
@@
 	8150 6650 8150 4150
 Text Notes 9100 6250 0    50   ~ 0
-U? acts as a comparator and\ngoes low  when Vin = 5.5V.\nInternal Vref = 2.495V
+Acts as a comparator and\ngoes low  when Vin = 5.5V.\nInternal Vref = 2.495V
 Wire Wire Line
 	10650 4900 10650 5650
 $Comp
-L Device:Q_PNP_BEC Q302
+L Device:Q_PNP_BEC Q802
 U 1 1 5F81D169
 P 9950 5250
-AR Path="/5F7CCAA0/5F81D169" Ref="Q302"  Part="1"
+AR Path="/5F7CCAA0/5F81D169" Ref="Q802"  Part="1"
 AR Path="/602C5383/5F81D169" Ref="Q?"  Part="1"
-F 0 "Q302" H 10141 5296 50  0000 L CNN
+F 0 "Q802" H 10141 5296 50  0000 L CNN
 F 1 "PMBT2907A" H 10141 5205 50  0000 L CNN
 F 2 "Package_TO_SOT_SMD:SOT-23_Handsoldering" H 10150 5350 50  0001 C CNN
@@
 Wire Notes Line style solid
 	10300 5950 10300 6300
+Text Label 6900 4600 0    50   ~ 0
+V_IN+_REV_PROTECTED
+Wire Wire Line
+	6250 4900 6250 6550
 $EndSCHEMATC

Commit message: Updated U801 DK link and part number, updated change log
Parts:
- U801: value TL432LI -> TL431LI; symbol irex_Reference_Voltage:TL432LI -> irex_Reference_Voltage:TL431LI; Digi-Key Link https://www.digikey.com/en/products/detail/texas-instruments/TL432LIACDBZR/9860322 -> https://www.digikey.com/en/products/detail/texas-instruments/TL431LIACDBZR/9861498; Digi-Key PN 296-53244-1-ND -> 296-53238-1-ND
Changed lines of the file:
@@
 	8350 5700 8850 5700
 $Comp
-L irex_Reference_Voltage:TL432LI U801
+L irex_Reference_Voltage:TL431LI U801
 U 1 1 5F7E207E
 P 8950 5700
@@
 AR Path="/602C5383/5F7E207E" Ref="U?"  Part="1"
 F 0 "U801" V 8996 5630 50  0000 R CNN
-F 1 "TL432LI" V 8905 5630 50  0000 R CNN
+F 1 "TL431LI" V 8905 5630 50  0000 R CNN
 F 2 "Package_TO_SOT_SMD:SOT-23" H 8950 5550 50  0001 C CIN
 F 3 "https://www.ti.com/lit/ds/symlink/tl431li.pdf?HQS=TI-null-null-digikeymode-df-pf-null-wwe&ts=1601074554367" H 8950 5700 50  0001 C CIN
-F 4 "https://www.digikey.com/en/products/detail/texas-instruments/TL432LIACDBZR/9860322" H 8950 5700 50  0001 C CNN "Digi-Key Link"
-F 5 "296-53244-1-ND" H 8950 5700 50  0001 C CNN "Digi-Key PN"
+F 4 "https://www.digikey.com/en/products/detail/texas-instruments/TL431LIACDBZR/9861498" H 8950 5700 50  0001 C CNN "Digi-Key Link"
+F 5 "296-53238-1-ND" H 8950 5700 50  0001 C CNN "Digi-Key PN"
 F 6 "TL432LI" H 8950 5700 50  0001 C CNN "MPN"
 	1    8950 5700
